File: PCB/HB-UNI-Sen-PM_v2p1.sch (EAGLE design)
At the start: 27 parts, among them IC1 MCP1700T-3302E_MB, IC3 MEGA8-AI, Q1 CSTCE, U1 CC1101SMD

Commit message: pcb silkscreen corrected in v2.1, first working version of software
Parts:
- removed JP1: IO, pinhead:PINHD-1X2
- removed JP2: I2C, pinhead:PINHD-1X4
- removed R2, R5: 10k, resistor:R-EU_R0805W
- added U$1: LOETKONTAKT4P, StephansLib:LOETKONTAKT4P
- S1: value SMDSWITCH6X4 -> CONFIG
Connections:
- removed net PC0: IC3.PC0(ADC0), R2.2
- removed net PC0DIV: JP1.1, R2.1, R5.2
- removed net PC1: IC3.PC1(ADC1), JP1.2
- net 3V3: now also U$1.4; no longer JP2.4
- net GND: now also U$1.3; no longer JP2.3, R5.1
- net SCL: now also U$1.2; no longer JP2.2
- net SDA: now also U$1.1; no longer JP2.1
Other:
- note added: "2.1"
- note removed: "1.0"
Changed lines of the file:
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@@
 <part name="R3" library="resistor" library_urn="urn:adsk.eagle:library:348" deviceset="R-EU_" device="R0805W" package3d_urn="urn:adsk.eagle:package:26060/1" value="220R"/>
 <part name="LED1" library="led" library_urn="urn:adsk.eagle:library:259" deviceset="LED" device="CHIPLED_0805" package3d_urn="urn:adsk.eagle:package:15821/2" value="gn"/>
-<part name="S1" library="StephansLib" deviceset="SMDSWITCH6X4" device=""/>
+<part name="S1" library="StephansLib" deviceset="SMDSWITCH6X4" device="" value="CONFIG"/>
 <part name="R1" library="resistor" library_urn="urn:adsk.eagle:library:348" deviceset="R-EU_" device="R0805W" package3d_urn="urn:adsk.eagle:package:26060/1" value="10k"/>
 <part name="C2" library="resistor" library_urn="urn:adsk.eagle:library:348" deviceset="C-EU" device="C0805K" package3d_urn="urn:adsk.eagle:package:26201/1" value="100n"/>
@@
 <part name="C5" library="resistor" library_urn="urn:adsk.eagle:library:348" deviceset="C-EU" device="C0805K" package3d_urn="urn:adsk.eagle:package:26201/1" value="100n"/>
 <part name="C8" library="resistor" library_urn="urn:adsk.eagle:library:348" deviceset="C-EU" device="C0805K" package3d_urn="urn:adsk.eagle:package:26201/1" value="100n"/>
-<part name="JP2" library="pinhead" library_urn="urn:adsk.eagle:library:325" deviceset="PINHD-1X4" device="" package3d_urn="urn:adsk.eagle:package:22407/2" value="I2C"/>
-<part name="JP1" library="pinhead" library_urn="urn:adsk.eagle:library:325" deviceset="PINHD-1X2" device="" package3d_urn="urn:adsk.eagle:package:22435/2" value="IO"/>
-<part name="R2" library="resistor" library_urn="urn:adsk.eagle:library:348" deviceset="R-EU_" device="R0805W" package3d_urn="urn:adsk.eagle:package:26060/1" value="10k"/>
-<part name="R5" library="resistor" library_urn="urn:adsk.eagle:library:348" deviceset="R-EU_" device="R0805W" package3d_urn="urn:adsk.eagle:package:26060/1" value="10k"/>
+<part name="U$1" library="StephansLib" deviceset="LOETKONTAKT4P" device=""/>
 </parts>
 <sheets>
 <sheet>
 <plain>
-<text x="246.38" y="-86.36" size="2.54" layer="94">1.0</text>
+<text x="246.38" y="-86.36" size="2.54" layer="94">2.1</text>
 <text x="154.94" y="-66.04" size="2.54" layer="94">(c) Stephan * CC by-nc-sa</text>
 </plain>
@@
 <instance part="C5" gate="G$1" x="-93.98" y="5.08"/>
 <instance part="C8" gate="G$1" x="-43.18" y="5.08"/>
-<instance part="JP2" gate="A" x="193.04" y="81.28"/>
-<instance part="JP1" gate="G$1" x="-48.26" y="-50.8"/>
-<instance part="R2" gate="G$1" x="-71.12" y="-38.1" rot="R90"/>
-<instance part="R5" gate="G$1" x="-71.12" y="-58.42" rot="R90"/>
+<instance part="U$1" gate="G$1" x="193.04" y="83.82" rot="R270"/>
 </instances>
 <busses>
@@
 <pinref part="SPS30" gate="A" pin="2"/>
 <wire x1="203.2" y1="86.36" x2="228.6" y2="86.36" width="0.1524" layer="91"/>
-<pinref part="JP2" gate="A" pin="1"/>
 <wire x1="190.5" y1="86.36" x2="149.86" y2="86.36" width="0.1524" layer="91"/>
 <junction x="149.86" y="86.36"/>
+<pinref part="U$1" gate="G$1" pin="1"/>
 </segment>
 </net>
@@
 <pinref part="SPS30" gate="A" pin="3"/>
 <wire x1="205.74" y1="83.82" x2="228.6" y2="83.82" width="0.1524" layer="91"/>
-<pinref part="JP2" gate="A" pin="2"/>
 <wire x1="190.5" y1="83.82" x2="147.32" y2="83.82" width="0.1524" layer="91"/>
 <junction x="147.32" y="83.82"/>
+<pinref part="U$1" gate="G$1" pin="2"/>
 </segment>
 </net>
@@
 <pinref part="C5" gate="G$1" pin="2"/>
 <pinref part="C8" gate="G$1" pin="2"/>
-<pinref part="JP2" gate="A" pin="3"/>
 <wire x1="190.5" y1="81.28" x2="180.34" y2="81.28" width="0.1524" layer="91"/>
 <wire x1="180.34" y1="81.28" x2="180.34" y2="-7.62" width="0.1524" layer="91"/>
@@
 <junction x="-109.22" y="-7.62"/>
 <label x="-111.76" y="-7.62" size="1.778" layer="95" rot="R180" xref="yes"/>
-</segment>
-<segment>
-<pinref part="R5" gate="G$1" pin="1"/>
-<wire x1="-71.12" y1="-63.5" x2="-71.12" y2="-66.04" width="0.1524" layer="91"/>
-<label x="-71.12" y="-66.04" size="1.778" layer="95" rot="R270" xref="yes"/>
+<pinref part="U$1" gate="G$1" pin="3"/>
 </segment>
 </net>
@@
 <junction x="5.08" y="53.34"/>
 <pinref part="C8" gate="G$1" pin="1"/>
-<pinref part="JP2" gate="A" pin="4"/>
 <wire x1="190.5" y1="78.74" x2="185.42" y2="78.74" width="0.1524" layer="91"/>
 <wire x1="185.42" y1="78.74" x2="185.42" y2="99.06" width="0.1524" layer="91"/>
+<pinref part="U$1" gate="G$1" pin="4"/>
 </segment>
 </net>
@@
 </segment>
 </net>
-<net name="PC0DIV" class="0">
-<segment>
-<pinref part="R2" gate="G$1" pin="1"/>
-<pinref part="R5" gate="G$1" pin="2"/>
-<wire x1="-71.12" y1="-43.18" x2="-71.12" y2="-48.26" width="0.1524" layer="91"/>
-<pinref part="JP1" gate="G$1" pin="1"/>
-<wire x1="-71.12" y1="-48.26" x2="-71.12" y2="-53.34" width="0.1524" layer="91"/>
-<wire x1="-50.8" y1="-48.26" x2="-71.12" y2="-48.26" width="0.1524" layer="91"/>
-<junction x="-71.12" y="-48.26"/>
-</segment>
-</net>
-<net name="PC0" class="0">
-<segment>
-<pinref part="R2" gate="G$1" pin="2"/>
-<wire x1="-71.12" y1="-33.02" x2="-71.12" y2="-30.48" width="0.1524" layer="91"/>
-<wire x1="-71.12" y1="-30.48" x2="-78.74" y2="-30.48" width="0.1524" layer="91"/>
-<label x="-78.74" y="-30.48" size="1.778" layer="95" rot="R180" xref="yes"/>
-</segment>
-<segment>
-<pinref part="IC3" gate="G$1" pin="PC0(ADC0)"/>
-<wire x1="58.42" y1="91.44" x2="60.96" y2="91.44" width="0.1524" layer="91"/>
-<label x="60.96" y="91.44" size="1.778" layer="95" xref="yes"/>
-</segment>
-</net>
-<net name="PC1" class="0">
-<segment>
-<pinref part="JP1" gate="G$1" pin="2"/>
-<wire x1="-50.8" y1="-50.8" x2="-78.74" y2="-50.8" width="0.1524" layer="91"/>
-<label x="-78.74" y="-50.8" size="1.778" layer="95" rot="R180" xref="yes"/>
-</segment>
-<segment>
-<pinref part="IC3" gate="G$1" pin="PC1(ADC1)"/>
-<wire x1="58.42" y1="88.9" x2="60.96" y2="88.9" width="0.1524" layer="91"/>
-<label x="60.96" y="88.9" size="1.778" layer="95" xref="yes"/>
-</segment>
-</net>
